File: board/beta.brd (EAGLE design)
At the start: 100 x 80 mm, 21 parts, among them IC1 W65C02S6TP, IC2-RAM CY62256LL-PC, IC7 74LS00N, IC8-ROM AT28C256-28DIP, IC9-PERIPHERALS W65C22S6TP

Commit message: completato pcb
Parts:
- added H1, H2: MOUNT-HOLE3.0, ITIS:3,0
- moved C6 3.49 mm to (77.2, 69.8)
- renumbered IC1 to IC1-CPU, IC7 to IC7-NAND, QG1 to QG1-XTAL
Routing:
- net VCC: track 0.00 -> 36.2 mm, vias 0 -> 1
- net GND: track 0.00 -> 27.5 mm, vias 0 -> 4
- added copper zone on layer 16, net GND
- added copper zone on layer 1, net VCC

Commit message: sistemato pcb
Parts:
- added U$1: LOGO-CYBERINDUSTRIES", CyberLibrary:LOGO-SMALL
- moved C6 1.35 mm to (76.2, 68.9)
- moved C5 1.27 mm to (20.6, 17.8)
- moved C4 0.95 mm to (88.9, 23.8)
- moved C3 0.63 mm to (10.8, 23.5)
Routing:
- net VCC: track 36.2 -> 35.2 mm
- net CS_RAM*: track 112.2 -> 112.9 mm
- net A15: track 87.2 -> 86.6 mm
Other:
- board text added: "+5V"
- board text added: "6502-computer <~ β v1.0 ~> CyberIndustries"
- board text added: "BOTTOM"
- board text added: "GND"
- board text added: "JLCJLCJLCJLC"
- board text added: "TOP"
Changed lines of the file:
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@@
 <wire x1="100" y1="80" x2="0" y2="80" width="0" layer="20"/>
 <wire x1="0" y1="80" x2="0" y2="0" width="0" layer="20"/>
+<text x="26.3525" y="53.975" size="1.778" layer="25">6502-computer
+&lt;~ β v1.0 ~&gt;
+CyberIndustries</text>
+<text x="11.43" y="50.8" size="1.27" layer="26" rot="MR270">JLCJLCJLCJLC</text>
+<text x="6.0325" y="72.0725" size="0.8128" layer="25" rot="R270">GND</text>
+<text x="6.0325" y="77.1525" size="0.8128" layer="25" rot="R270">+5V</text>
+<text x="10.4775" y="78.105" size="0.8128" layer="1">TOP</text>
+<text x="13.97" y="78.105" size="0.8128" layer="16" rot="MR0">BOTTOM</text>
 </plain>
 <attributes>
@@
 <attribute name="NAME" x="28.8925" y="31.496" size="1.27" layer="25" ratio="10"/>
 </element>
-<element name="C3" library="ITIS" package="E2-5" value="1uF" x="10.795" y="24.13" smashed="yes">
-<attribute name="NAME" x="9.8425" y="20.066" size="1.27" layer="25" ratio="10"/>
-</element>
-<element name="C4" library="ITIS" package="E2-5" value="1uF" x="88.9" y="24.765" smashed="yes">
-<attribute name="NAME" x="89.8525" y="21.844" size="1.27" layer="25" ratio="10" rot="R180"/>
-</element>
-<element name="C5" library="ITIS" package="E2-5" value="1uF" x="21.9075" y="17.78" smashed="yes" rot="R90">
-<attribute name="NAME" x="22.86" y="14.859" size="1.27" layer="25" ratio="10" rot="R180"/>
-</element>
-<element name="C6" library="ITIS" package="E2-5" value="1uF" x="77.1525" y="69.85" smashed="yes" rot="R90">
-<attribute name="NAME" x="74.93" y="68.5165" size="1.27" layer="25" ratio="10" rot="R180"/>
+<element name="C3" library="ITIS" package="E2-5" value="1uF" x="10.795" y="23.495" smashed="yes">
+<attribute name="NAME" x="9.8425" y="19.431" size="1.27" layer="25" ratio="10"/>
+</element>
+<element name="C4" library="ITIS" package="E2-5" value="1uF" x="88.9" y="23.8125" smashed="yes">
+<attribute name="NAME" x="89.8525" y="20.8915" size="1.27" layer="25" ratio="10" rot="R180"/>
+</element>
+<element name="C5" library="ITIS" package="E2-5" value="1uF" x="20.6375" y="17.78" smashed="yes" rot="R90">
+<attribute name="NAME" x="21.59" y="14.859" size="1.27" layer="25" ratio="10" rot="R180"/>
+</element>
+<element name="C6" library="ITIS" package="E2-5" value="1uF" x="76.2" y="68.8975" smashed="yes" rot="R90">
+<attribute name="NAME" x="73.9775" y="67.564" size="1.27" layer="25" ratio="10" rot="R180"/>
 </element>
 <element name="POW" library="CiniTechLibrary" package="AK500-2" package3d_urn="urn:adsk.eagle:package:17855270/2" value="AK500" x="2.54" y="76.2" smashed="yes" rot="R270">
-<attribute name="NAME" x="6.54" y="76.2" size="1.27" layer="25" rot="R270"/>
+<attribute name="NAME" x="7.81" y="75.8825" size="1.27" layer="25" rot="R270"/>
 </element>
 <element name="H1" library="ITIS" package="3,0" value="MOUNT-HOLE3.0" x="5.08" y="9.8425" smashed="yes"/>
 <element name="H2" library="ITIS" package="3,0" value="MOUNT-HOLE3.0" x="72.0725" y="74.93" smashed="yes"/>
+<element name="U$1" library="CyberLibrary" package="LOGO-SMALL" value="LOGO-CYBERINDUSTRIES&quot;" x="86.6775" y="7.9375" smashed="yes"/>
 </elements>
 <signals>
@@
 </polygon>
 <wire x1="5.715" y1="15.875" x2="7.9375" y2="18.0975" width="0.6096" layer="16"/>
-<wire x1="7.9375" y1="18.0975" x2="7.9375" y2="22.86" width="0.6096" layer="16"/>
-<wire x1="7.9375" y1="22.86" x2="9.2075" y2="24.13" width="0.6096" layer="16"/>
-<wire x1="9.2075" y1="24.13" x2="9.779" y2="24.13" width="0.6096" layer="16"/>
+<wire x1="7.9375" y1="18.0975" x2="7.9375" y2="21.59" width="0.6096" layer="16"/>
+<wire x1="9.779" y1="23.495" x2="9.779" y2="23.4315" width="0.6096" layer="16"/>
+<wire x1="9.779" y1="23.4315" x2="7.9375" y2="21.59" width="0.6096" layer="16"/>
 <wire x1="81.28" y1="31.115" x2="81.28" y2="28.575" width="0.6096" layer="16"/>
 <wire x1="36.195" y1="50.4825" x2="36.195" y2="67.31" width="0.6096" layer="16"/>
@@
 <wire x1="13.335" y1="68.58" x2="10.795" y2="66.04" width="0.1524" layer="16"/>
 <wire x1="22.225" y1="68.58" x2="13.335" y2="68.58" width="0.1524" layer="16"/>
-<wire x1="88.9" y1="7.62" x2="72.39" y2="7.62" width="0.1524" layer="16"/>
-<wire x1="88.9" y1="69.5325" x2="88.9" y2="7.62" width="0.1524" layer="16"/>
+<wire x1="88.9" y1="69.5325" x2="88.9" y2="8.5725" width="0.1524" layer="16"/>
+<wire x1="88.9" y1="8.5725" x2="88.265" y2="7.9375" width="0.1524" layer="16"/>
+<wire x1="72.0725" y1="7.9375" x2="88.265" y2="7.9375" width="0.1524" layer="16"/>
 </signal>
 <signal name="N$1">
@@
 <wire x1="52.705" y1="49.2125" x2="51.435" y2="50.4825" width="0.1524" layer="1"/>
 <wire x1="4.445" y1="62.23" x2="3.175" y2="60.96" width="0.1524" layer="1"/>
-<wire x1="80.645" y1="62.23" x2="51.435" y2="62.23" width="0.1524" layer="1"/>
-<wire x1="51.435" y1="62.23" x2="4.445" y2="62.23" width="0.1524" layer="1"/>
+<wire x1="80.645" y1="62.23" x2="52.07" y2="62.23" width="0.1524" layer="1"/>
+<wire x1="52.07" y1="62.23" x2="4.445" y2="62.23" width="0.1524" layer="1"/>
 <wire x1="81.28" y1="61.595" x2="80.645" y2="62.23" width="0.1524" layer="1"/>
 <wire x1="51.435" y1="60.325" x2="51.435" y2="50.4825" width="0.1524" layer="16"/>
-<wire x1="51.435" y1="62.23" x2="51.435" y2="60.325" width="0.1524" layer="1"/>
 <via x="51.435" y="60.325" extent="1-16" drill="0.35"/>
+<wire x1="51.435" y1="60.325" x2="51.435" y2="61.595" width="0.1524" layer="1"/>
+<wire x1="51.435" y1="61.595" x2="52.07" y2="62.23" width="0.1524" layer="1"/>
 </signal>
 <signal name="D2">
@@
 <contactref element="IC2-RAM" pad="7"/>
 <contactref element="IC8-ROM" pad="23"/>
-<wire x1="15.24" y1="43.18" x2="18.415" y2="43.18" width="0.1524" layer="16"/>
-<wire x1="15.24" y1="55.245" x2="15.24" y2="43.18" width="0.1524" layer="16"/>
+<wire x1="15.24" y1="55.245" x2="15.24" y2="43.815" width="0.1524" layer="16"/>
 <wire x1="17.145" y1="57.15" x2="15.24" y2="55.245" width="0.1524" layer="16"/>
 <wire x1="20.32" y1="57.15" x2="17.145" y2="57.15" width="0.1524" layer="16"/>
@@
 <via x="20.955" y="56.515" extent="1-16" drill="0.35"/>
 <via x="77.47" y="55.88" extent="1-16" drill="0.35"/>
+<wire x1="15.24" y1="43.815" x2="15.875" y2="43.18" width="0.1524" layer="16"/>
+<wire x1="15.875" y1="43.18" x2="18.415" y2="43.18" width="0.1524" layer="16"/>
 </signal>
 <signal name="A12">
@@
 <contactref element="IC7-NAND" pad="2"/>
 <contactref element="IC9-PERIPHERALS" pad="23"/>
-<wire x1="83.82" y1="69.85" x2="81.28" y2="69.85" width="0.1524" layer="1"/>
-<wire x1="81.28" y1="69.85" x2="81.28" y2="69.5325" width="0.1524" layer="1"/>
-<wire x1="83.82" y1="69.85" x2="83.82" y2="69.5325" width="0.1524" layer="1"/>
 <wire x1="70.485" y1="26.67" x2="69.215" y2="25.4" width="0.1524" layer="16"/>
 <wire x1="70.485" y1="51.435" x2="70.485" y2="29.21" width="0.1524" layer="16"/>
@@
 <wire x1="64.135" y1="55.245" x2="66.675" y2="55.245" width="0.1524" layer="16"/>
 <wire x1="64.135" y1="50.4825" x2="64.135" y2="55.245" width="0.1524" layer="16"/>
-<wire x1="76.835" y1="64.77" x2="81.28" y2="69.215" width="0.1524" layer="16"/>
-<wire x1="76.835" y1="35.56" x2="76.835" y2="64.77" width="0.1524" layer="16"/>
-<wire x1="70.485" y1="29.21" x2="76.835" y2="35.56" width="0.1524" layer="16"/>
-<wire x1="81.28" y1="69.215" x2="81.28" y2="69.5325" width="0.1524" layer="16"/>
+<wire x1="76.5175" y1="35.2425" x2="76.5175" y2="64.77" width="0.1524" layer="16"/>
+<wire x1="70.485" y1="29.21" x2="76.5175" y2="35.2425" width="0.1524" layer="16"/>
+<wire x1="76.5175" y1="64.77" x2="81.28" y2="69.5325" width="0.1524" layer="16"/>
+<wire x1="81.28" y1="69.5325" x2="83.82" y2="69.5325" width="0.1524" layer="16"/>
 </signal>
 <signal name="A15*">
@@
 <wire x1="1.905" y1="65.405" x2="1.27" y2="64.77" width="0.1524" layer="1"/>
 <wire x1="1.27" y1="64.77" x2="1.27" y2="50.165" width="0.1524" layer="1"/>
-<wire x1="90.17" y1="65.405" x2="1.905" y2="65.405" width="0.1524" layer="1"/>
-<wire x1="93.98" y1="69.215" x2="90.17" y2="65.405" width="0.1524" layer="1"/>
-<wire x1="93.98" y1="69.215" x2="93.98" y2="69.5325" width="0.1524" layer="1"/>
+<wire x1="91.44" y1="65.405" x2="1.905" y2="65.405" width="0.1524" layer="1"/>
+<wire x1="93.98" y1="67.945" x2="91.44" y2="65.405" width="0.1524" layer="1"/>
+<wire x1="93.98" y1="67.945" x2="93.98" y2="69.5325" width="0.1524" layer="1"/>
 </signal>
 <signal name="CA1">
@@
 </drawing>
 <compatibility>
+<note version="6.3" minversion="6.2.2" severity="warning">
+Since Version 6.2.2 text objects can contain more than one line,
+which will not be processed correctly with this version.
+</note>
 <note version="8.2" severity="warning">
 Since Version 8.2, EAGLE supports online libraries. The ids
