File: board/beta.sch (EAGLE design)
At the start: 21 parts, among them IC1 W65C02S6TP, IC2-RAM CY62256LL-PC, IC7 74LS00N, IC8-ROM AT28C256-28DIP, IC9-PERIPHERALS W65C22S6TP

Commit message: completato pcb
Parts:
- added H1, H2: MOUNT-HOLE3.0, ITIS:MOUNT-HOLE3.0
- renumbered IC1 to IC1-CPU, IC7 to IC7-NAND, QG1 to QG1-XTAL

Commit message: sistemato pcb
Parts:
- added U$1: LOGO-CYBERINDUSTRIES", CyberLibrary:LOGO-CYBERINDUSTRIES"
Changed lines of the file:
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@@
 <part name="H1" library="ITIS" deviceset="MOUNT-HOLE" device="3.0"/>
 <part name="H2" library="ITIS" deviceset="MOUNT-HOLE" device="3.0"/>
+<part name="U$1" library="CyberLibrary" deviceset="LOGO-CYBERINDUSTRIES" device="&quot;"/>
 </parts>
 <sheets>
@@
 <attribute name="VALUE" x="19.812" y="-60.8838" size="1.778" layer="96"/>
 </instance>
+<instance part="U$1" gate="G$1" x="55.88" y="-55.88" smashed="yes"/>
 </instances>
 <busses>
